File: pcb/rev1/cert3d_rev1.sch (EAGLE design)
At the start: 94 parts, among them J1 CONN2TSW-S, J10 CONN2TSW-S, J11 CONN2TSW-S, J12 CONN10CNC-3220-10-0100-00, J13 USB-5PINTOPVIA, J14 CONN4TSW-S, J15 CONN4TSW-S, J16 CONN4TSW-S, J17 CONN2TSW-S, J2 CONN2TSW-S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

Commit message: updated eagle board files with part numbers
Parts:
- C10, C5, C6, C7, C8, C9: PN (none) -> C0805C104K5RACTU
- C3, C4: PN (none) -> C0805C225K3RAC7800
- LED1: PN (none) -> 150080GS75000
- LED2: PN (none) -> 150080RS75000
- U1: PN (none) -> STM32F405RGT6‎
- Y1: PN (none) -> FC4STCBMF8.0-BAG200
Other:
- moved on the sheet: C1, C10, C13, C15, C16, C17, C2, C3, C4, C5, C6, C7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
