File: pcb/rev2/cert3d_rev2.brd (EAGLE design)
At the start: 69.8 x 48.3 mm, 76 parts, among them J1 CONN4TSW-S, J10 CONN4TSW-S, J11 CONN4TSW-S, J12 CONN4TSW-S, J13 CONN4TSW-S, J14 CONN4TSW-S, J15 CONN4TSW-S, J16 CONN4TSW-S, J17 USB-5PINTOPVIA, J18 STLINK-V3/SWDCNC-3220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

Commit message: finalized rev2 PWB
Routing:
- net GND: track 82.2 -> 81.5 mm
- net +3V3: track 226.8 -> 227.3 mm
Changed lines of the file:
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@@
 <drawing>
 <settings>
-<setting alwaysvectorfont="yes"/>
+<setting alwaysvectorfont="no"/>
 <setting verticaltext="up"/>
 </settings>
@@
 <wire x1="34.671" y1="3.429" x2="34.798" y2="3.556" width="0.254" layer="1"/>
 <wire x1="24.257" y1="3.81" x2="25.527" y2="3.81" width="0.254" layer="1"/>
-<via x="32.258" y="15.875" extent="1-16" drill="0.3302"/>
-<via x="34.544" y="13.462" extent="1-16" drill="0.3302"/>
-<wire x1="30.596290625" y1="15.1609125" x2="31.310378125" y2="15.875" width="0.254" layer="1"/>
-<wire x1="31.310378125" y1="15.875" x2="32.258" y2="15.875" width="0.254" layer="1"/>
-<wire x1="33.778271875" y1="11.97893125" x2="34.544" y2="12.744659375" width="0.254" layer="1"/>
-<wire x1="34.544" y1="12.744659375" x2="34.544" y2="13.462" width="0.254" layer="1"/>
+<via x="31.877" y="16.129" extent="1-16" drill="0.3302"/>
+<via x="34.798" y="13.335" extent="1-16" drill="0.3302"/>
+<wire x1="30.596290625" y1="15.1609125" x2="31.564378125" y2="16.129" width="0.254" layer="1"/>
+<wire x1="31.564378125" y1="16.129" x2="31.877" y2="16.129" width="0.254" layer="1"/>
+<wire x1="33.778271875" y1="11.97893125" x2="34.798" y2="12.998659375" width="0.254" layer="1"/>
+<wire x1="34.798" y1="12.998659375" x2="34.798" y2="13.335" width="0.254" layer="1"/>
 <via x="40.132" y="8.128" extent="1-16" drill="0.3302"/>
-<via x="44.831" y="9.017" extent="1-16" drill="0.3302"/>
-<via x="48.514" y="12.573" extent="1-16" drill="0.3302"/>
-<via x="51.054" y="15.113" extent="1-16" drill="0.3302"/>
+<via x="45.212" y="9.398" extent="1-16" drill="0.3302"/>
+<via x="48.895" y="13.081" extent="1-16" drill="0.3302"/>
+<via x="51.308" y="15.621" extent="1-16" drill="0.3302"/>
 <via x="53.213" y="17.272" extent="1-16" drill="0.3302"/>
 <wire x1="54.637921875" y1="16.575125" x2="53.941046875" y2="17.272" width="0.254" layer="1"/>
 <wire x1="53.941046875" y1="17.272" x2="53.213" y2="17.272" width="0.254" layer="1"/>
-<wire x1="52.5166" y1="14.453803125" x2="51.857403125" y2="15.113" width="0.254" layer="1"/>
-<wire x1="51.857403125" y1="15.113" x2="51.054" y2="15.113" width="0.254" layer="1"/>
-<wire x1="50.041725" y1="11.97893125" x2="49.44765625" y2="12.573" width="0.254" layer="1"/>
-<wire x1="49.44765625" y1="12.573" x2="48.514" y2="12.573" width="0.254" layer="1"/>
-<wire x1="46.50619375" y1="8.443396875" x2="45.932590625" y2="9.017" width="0.254" layer="1"/>
-<wire x1="45.932590625" y1="9.017" x2="44.831" y2="9.017" width="0.254" layer="1"/>
+<wire x1="52.5166" y1="14.453803125" x2="51.349403125" y2="15.621" width="0.254" layer="1"/>
+<wire x1="51.349403125" y1="15.621" x2="51.308" y2="15.621" width="0.254" layer="1"/>
+<wire x1="50.041725" y1="11.97893125" x2="48.93965625" y2="13.081" width="0.254" layer="1"/>
+<wire x1="48.93965625" y1="13.081" x2="48.895" y2="13.081" width="0.254" layer="1"/>
+<wire x1="46.50619375" y1="8.443396875" x2="45.551590625" y2="9.398" width="0.254" layer="1"/>
+<wire x1="45.551590625" y1="9.398" x2="45.212" y2="9.398" width="0.254" layer="1"/>
 <wire x1="39.081571875" y1="6.67563125" x2="40.132" y2="7.726059375" width="0.254" layer="1"/>
 <wire x1="40.132" y1="7.726059375" x2="40.132" y2="8.128" width="0.254" layer="1"/>
@@
 <wire x1="64.516" y1="11.43" x2="62.23" y2="11.43" width="0.254" layer="1"/>
 <wire x1="62.23" y1="11.43" x2="60.96" y2="12.7" width="0.254" layer="1"/>
+<wire x1="60.96" y1="12.7" x2="60.96" y2="17.653" width="0.254" layer="1"/>
 <wire x1="60.96" y1="17.653" x2="59.817" y2="18.796" width="0.254" layer="1"/>
-<wire x1="60.96" y1="12.7" x2="60.96" y2="17.653" width="0.254" layer="1"/>
-<wire x1="59.817" y1="18.796" x2="53.34" y2="18.796" width="0.254" layer="1"/>
-<wire x1="53.34" y1="18.796" x2="52.832" y2="18.796" width="0.254" layer="1"/>
+<wire x1="59.817" y1="18.796" x2="52.832" y2="18.796" width="0.254" layer="1"/>
 </signal>
 <signal name="USB_HS_DM">
@@
 <wire x1="26.289" y1="19.05" x2="26.289" y2="17.399" width="0.254" layer="1"/>
 <wire x1="26.289" y1="17.399" x2="27.813" y2="15.875" width="0.254" layer="1"/>
-<wire x1="33.655" y1="16.764" x2="35.941" y2="14.478" width="0.254" layer="1"/>
-<wire x1="31.492271875" y1="16.764" x2="30.2427375" y2="15.514465625" width="0.254" layer="1"/>
-<wire x1="33.655" y1="16.764" x2="31.492271875" y2="16.764" width="0.254" layer="1"/>
+<wire x1="33.401" y1="17.018" x2="35.941" y2="14.478" width="0.254" layer="1"/>
+<wire x1="31.746271875" y1="17.018" x2="30.2427375" y2="15.514465625" width="0.254" layer="1"/>
+<wire x1="33.401" y1="17.018" x2="31.746271875" y2="17.018" width="0.254" layer="1"/>
 <wire x1="35.941" y1="14.478" x2="35.941" y2="13.434553125" width="0.254" layer="1"/>
 <wire x1="35.941" y1="13.434553125" x2="34.131825" y2="11.625378125" width="0.254" layer="1"/>
@@
 <wire x1="40.894" y1="8.636" x2="41.021" y2="8.763" width="0.254" layer="1"/>
 <wire x1="42.545" y1="8.763" x2="41.021" y2="8.763" width="0.254" layer="16"/>
-<wire x1="46.859746875" y1="8.79695" x2="45.750696875" y2="9.906" width="0.254" layer="1"/>
-<wire x1="43.688" y1="9.906" x2="42.545" y2="8.763" width="0.254" layer="1"/>
-<wire x1="45.750696875" y1="9.906" x2="43.688" y2="9.906" width="0.254" layer="1"/>
+<wire x1="46.859746875" y1="8.79695" x2="45.369696875" y2="10.287" width="0.254" layer="1"/>
+<wire x1="44.069" y1="10.287" x2="42.545" y2="8.763" width="0.254" layer="1"/>
+<wire x1="45.369696875" y1="10.287" x2="44.069" y2="10.287" width="0.254" layer="1"/>
 <wire x1="41.021" y1="8.763" x2="38.481" y2="11.303" width="0.254" layer="16"/>
 <wire x1="38.481" y1="11.303" x2="38.481" y2="11.811" width="0.254" layer="16"/>
